File: justadistancemeasurer/justadistancemeasurer.kicad_sch (KiCad schematic)
At the start: 0 parts

Commit message: .
Parts:
- added BT1: Battery, symbol Device:Battery
- added SW1: SW_Push, symbol Switch:SW_Push
- added U1: HC-SR04, HC-SR04:XCVR_HC-SR04, symbol HC-SR04:HC-SR04
- added U2: XIAO-RP2040-DIP, Module:MOUDLE14P-XIAO-DIP-SMD, symbol Seeed_Studio_XIAO_Series:XIAO-RP2040-DIP
Connections:
- new net: BT1.1 (+), SW1.1
- new net GND: BT1.2 (-), U1.2 (GND), U2.13 (GND)
- new net Power: SW1.2, U1.1 (VCC), U2.14 (VBUS)
- new net RX: U1.3 (RX), U2.8 (GPIO1/RX)
- new net TX: U1.4 (TX), U2.7 (GPIO0/TX)
